File: slouchpad_pcb/slouchpad_v1_leftpad.sch (EAGLE design)
At the start: 47 parts, among them U2 MIC5219, U3 ATMEGA32U4, Y1 16MHz

Commit message: Retooled the project to be a modular joypad
Rather than being a shield for the SparkFun Pro Micro Arduino, the slouchpad will simply be a modular joypad for use with any microcontroller.

Modified the license to reflect the removal of the SparkFun Pro Micro

Removed backup design files

Created button layout for left thumb pad

Modified all board positions to units of mm where possible.

Signed-off-by: Eric Jones <eric.r.k.jones@gmail.com>
Parts:
- removed C1, C3: 0.1uF, SparkFun:CAP0603-CAP
- removed C10, C5, C6: 1uF, SparkFun:CAP0603-CAP
- removed C13, C19: 10uF, SparkFun:CAP_POL1206
- removed C2, C4: 22pF, SparkFun:CAP0603-CAP
- removed D1: Yellow, SparkFun:LED0603
- removed D2: (no value), SparkFun:DIODESOD
- removed D3: Green, SparkFun:LED0603
- removed F1: 500mA, SparkFun:PTCSMD
- removed FRAME1: FRAME-LETTER, SparkFun-Aesthetics:FRAME-LETTER
- removed JP3: (no value), pinhead:PINHD-1X3
- removed JP4: (no value), pinhead:PINHD-1X13
- removed JP6, JP7: M12PTH, SparkFun:M12PTH
- removed LED1: Red, SparkFun:LED0603
- removed R10: 10K, resistor:R-US_M1206
- removed R11: 1K, SparkFun:RESISTOR0603-RES
- removed R5, R7: 22, SparkFun:RESISTOR0603-RES
- removed R6: 330, SparkFun:RESISTOR0603-RES
- removed R8: 33K, resistor:R-US_M1206
- removed R9: 47K, resistor:R-US_M1206
- removed SJ1: Closed for 5V Board, SparkFun:SOLDERJUMPERNC
- removed U$1: LOGO-SFESK, SparkFun:LOGO-SFESK
- removed U$11: LOGO-SFENEW, SparkFun:LOGO-SFENEW
- removed U$3: OSHW-LOGOS, SparkFun:OSHW-LOGOS
- removed U2: MIC5219, SparkFun:V_REG_LDOSMD
- removed U3: ATMEGA32U4, Testing:ATMEGA32U4OUTFAKES
- removed X1: (no value), Testing:USB-ABIN&OUT
- removed Y1: 16MHz, SparkFun:CRYSTAL5X3
- JP1: value FIDUCIALUFIDUCIAL -> (none); device SparkFun:FIDUCIALUFIDUCIAL -> pinhead:PINHD-1X13
- JP2: value FIDUCIALUFIDUCIAL -> (none); device SparkFun:FIDUCIALUFIDUCIAL -> pinhead:PINHD-1X3
- R1: value 10K -> (none); device resistor:R-US_M1206 -> resistor:R-US_0204/5
- R2: value 10K -> (none); device SparkFun:RESISTOR0603-RES -> resistor:R-US_0204/5
- R3: value 22K -> (none); device resistor:R-US_M1206 -> resistor:R-US_0204/5
- R4: value 330 -> (none); device SparkFun:RESISTOR0603-RES -> resistor:R-US_0204/5
Connections:
- removed net A0: DOWN.2, JP6.8, LEFT.2, R10.1, RIGHT.2, U3.PF7(ADC7), UP.2
- removed net A1: JOY1X.S, JP6.7, U3.PF6(ADC6)
- removed net A2: JOY1Y.S, JP6.6, U3.PF5(ADC5)
- removed net A3: JP6.5, U3.PF4(ADC4)
- removed net A4: U3.PF1(ADC1)
- removed net A5: U3.PF0(ADC0)
- removed net AREF: C1.2, U3.AREF
- removed net D+: R5.1, U3.D+
- removed net D-: R7.1, U3.D-
- removed net D10: JP6.12, U3.PB6(ADC13)
- removed net D11: U3.PB7
- removed net D12: U3.PD6(ADC9)
- removed net D13: U3.PC7
- removed net D14: R4.1, U3.PB3(MISO)
- removed net D2: JP7.8, U3.PD1(SDA)
- removed net D3: JP7.7, U3.PD0(SCL)
- removed net D4: JP7.6, U3.PD4(ADC8)
- removed net D5: JP7.5, U3.PC6
- removed net D6: JP7.4, U3.PD7(ADC10)
- removed net D7: JP7.3, U3.PE6
- removed net D8: JP7.2, U3.PB4(ADC11)
- removed net D9: JP7.1, U3.PB5(ADC12)
- removed net MISO: JP6.10, U3.PB0(SS)
- removed net MOSI: JP6.11, U3.PB2(MOSI)
- removed net N$1: C4.1, U3.XTAL2, Y1.1
- removed net N$10: DOWN.1, R3.1
- removed net N$11: LEFT.1, R8.1
- removed net N$12: R9.1, RIGHT.1
- removed net N$14: SELECT.2
- removed net N$15: MENU.2
- removed net N$38: LED1.A, R11.1
- removed net N$4: C5.2, U3.UCAP
- removed net N$5: D1.C, R4.2
- removed net N$6: R7.2, X1.D-
- removed net N$7: D3.C, R6.2
- removed net N$8: R5.2, X1.D+
- removed net N$9: R1.1, UP.1
- removed net RAW: C19.+, D2.C, JP6.1, U2.EN, U2.IN
- removed net RESET: JP6.3, R2.1, U3.!RESET
- removed net RXI: JP7.11, U3.PD2(RX)
- removed net SCK: JP6.9, U3.PB1(SCK)
- removed net TXLED: R6.1, U3.PD5
- removed net TXO: JP7.12, U3.PD3(TX)
- removed net UVCC: C6.2, F1.1, U3.UVCC, U3.VBUS, X1.VBUS
- new net A: JP1.7
- new net B: JP1.8
- new net C: JP1.9
- new net DOWN: DOWN.1, R2.2
- new net JOYX: JOY1X.S, JP1.12
- new net JOYY: JOY1Y.S, JP1.10
- new net LEFT: LEFT.1, R3.2
- new net MENU: MENU.1
- new net RIGHT: R4.2, RIGHT.1
- new net SELECT: SELECT.1
- new net START: JP1.1
- new net UP: R1.2, UP.1
- new net X: JP1.6
- new net Y: JP1.5
- new net Z: JP1.4
- net GND: now also DOWN.2, JP1.13, JP2.2, LEFT.2, MENU.2, RIGHT.2, SELECT.2, UP.2; no longer C1.1, C10.2, C13.-, C19.-, C2.2, C3.1, C4.2, C5.1, C6.1, JP6.2, JP7.10, JP7.9, LED1.C, MENU.1, R1.2, R3.2, R8.2, R9.2, SELECT.1, U2.GND, U3.GND@15, U3.GND@23, U3.GND@35, U3.GND@43, U3.PE2/!HWB, U3.UGND, X1.GND
- net N$2: now also JP1.2, JP2.1; no longer C2.1, U3.XTAL1, Y1.2
- net N$3: now also JP1.3, JP2.3; no longer D2.A, F1.2, SJ1.1
- net VCC: now also JP1.11; no longer C10.1, C13.+, C3.2, D1.A, D3.A, JP6.4, R10.2, R11.2, R2.2, SJ1.2, U2.OUT, U3.AVCC@24, U3.AVCC@44, U3.VCC@14, U3.VCC@34
Other:
- note removed: "Added fuse and diode protection"
- note removed: "Added two small squares of tRestrict to keep the ground plane away from the sides of IC legs"
- note removed: "Arduino Pro Mini Design by Spark Fun Electronics"
- note removed: "Board is marked with combination of"
- note removed: "Change to 500mA regulator"
- note removed: "Changed LEDs to be tied to VCC"
- note removed: "Changes on v1.1:"
- note removed: "Changes on v1.2:"
- note removed: "Changes on v1.3:"
- note removed: "Corrected silk on D14"
- note removed: "Max Current Output: 500mA"
- note removed: "Max Voltage Input: 16VDC"
- note removed: "Not used"
- note removed: "Open for 3.3V Board"
- note removed: "Original Arduino Mini Design by Team Arduino"
- note removed: "Pro Micro Design by Spark Fun Electronics"
- note removed: "Renamed SS net to D14 (from D17)"
- note removed: "Routed directly inward or outward from each leg on the IC"
- note removed: "Updated QFN package on 32U4 to be 1:1"
- note removed: "Updated package on USB micro B (2 new pads)"
- note removed: "Updated symbol of 32U4 in schematic (switched MISO and SS placement)"
- note removed: "VCC = 5V or 3.3V Output"
- note removed: "resonator frequency and regulator voltage."
- note removed: "v13"

Commit message: Finished board layouts
Cleaned up schematics
Parts:
- added R5: 10K, resistor:R-US_0204/5
- JP1: device pinhead:PINHD-1X13 -> pinhead:PINHD-1X9
- R1: value (none) -> 10K
- R2: value (none) -> 22K
- R3: value (none) -> 33K
- R4: value (none) -> 47K
Connections:
- removed net A: JP1.7
- removed net B: JP1.8
- removed net C: JP1.9
- removed net DOWN: DOWN.1, R2.2
- removed net LEFT: LEFT.1, R3.2
- removed net RIGHT: R4.2, RIGHT.1
- removed net START: JP1.1
- removed net UP: R1.2, UP.1
- removed net X: JP1.6
- removed net Y: JP1.5
- removed net Z: JP1.4
- new net DPAD: JP1.8, R1.1, R2.1, R3.1, R4.1, R5.2
- new net N$1: JP1.2, JP2.3
- new net N$4: R3.2, RIGHT.1
- new net N$5: DOWN.1, R4.2
- new net N$6: R2.2, UP.1
- net GND: now also JP1.9; no longer JP1.13
- net JOYX: now also JP1.7; no longer JP1.12
- net JOYY: now also JP1.5; no longer JP1.10
- net MENU: now also JP1.4
- net N$2: now also JP1.3; no longer JP1.2
- net N$3: now also LEFT.1, R1.2; no longer JP1.3, JP2.3
- net SELECT: now also JP1.1
- net VCC: now also JP1.6, R5.1; no longer JP1.11
